File: Fuente_Conmutada.kicad_sch (KiCad schematic)
At the start: 48 parts, among them J1 Terminal_220v, J2 Terminal_12v, J3 Vout, Q1 IRF840, Q2 IRF840, T1 Transformer_1P_SS, U1 TL494, U2 IR2110

Commit message: dad
Parts:
- removed JP9: Jumper, Connector_PinHeader_2.54mm:PinHeader_1x02_P2.54mm_Vertical, symbol Jumper:Jumper_2_Bridged
Connections:
- net LO: now reaches D4.1 (K), R10.1
- net LO: now also JP6.2 (B)
- net Vref: now reaches U1.13 (OUTCTRL)
- net Vref: now also R3.1, R5.1, U1.14 (REF), U1.15 (2IN-), U1.2 (1IN-)
- net Vs: now reaches C4.2, C5.2, U2.5 (VS)
- net Vs: now also JP7.1 (A), Q1.3 (S), Q2.2 (D), R12.1
- net at T1.3 (SA): now also D5.3 (A2)
- net at D3.2 (A), Q1.1 (G), R9.2: now also R12.2; no longer R12.1
- net PWM1: now reaches U2.10 (HIN)
- net PWM1: now also JP3.2 (B)
- net PWM2: now reaches U2.12 (LIN)
- net PWM2: now also JP4.2 (B)
- net VAC: now reaches F1.2, J1.2 (Pin_2)
- net HO: now reaches D3.1 (K), R9.1
- net HO: now also JP5.2 (B)
- net 1 renamed GND
- new net Punto_medio: JP2.2 (B), R13.2, T1.2 (AB)
Other:
- moved on the sheet: JP2, JP5, R12
